Commit message: Update

File: go2_description/xacro/go2.xacro (robot description, xacro)
@@ -5,7 +5,7 @@
      For more information, please see http://wiki.ros.org/sw_urdf_exporter -->
 <robot
-  name="go2_description">
-  <link
-    name="base">
+  name="go2_description" xmlns:xacro="http://ros.org/wiki/xacro">
+  <link
+    name="base_link">
     <inertial>
       <origin
@@ -28,5 +28,5 @@
       <geometry>
         <mesh
-          filename="package://go2_description/dae/base.dae" />
+          filename="file://$(find go2_description)/dae/base_link.dae" />
       </geometry>
       <material
@@ -43,4 +43,18 @@
     </collision>
   </link>
+    <!-- 添加虚拟根链接 -->
+    <link name="dummy_base_link">
+        <visual>
+            <geometry>
+                <box size="0.001 0.001 0.001"/> <!-- 极小尺寸 -->
+            </geometry>
+        </visual>
+    </link>
+    <!-- 添加固定关节连接虚拟链接和原base_link -->
+    <joint name="dummy_joint" type="fixed">
+        <parent link="dummy_base_link"/>
+        <child link="base_link"/>
+        <origin xyz="0 0 0" rpy="0 0 0"/>
+    </joint>
   <link
     name="Head_upper">
@@ -75,5 +89,5 @@
       rpy="0 0 0" />
     <parent
-      link="base" />
+      link="base_link" />
     <child
       link="Head_upper" />
@@ -141,5 +155,5 @@
       <geometry>
         <mesh
-          filename="package://go2_description/dae/hip.dae" />
+          filename="file://$(find go2_description)/dae/hip.dae" />
       </geometry>
       <material
@@ -163,5 +177,5 @@
       rpy="0 0 0" />
     <parent
-      link="base" />
+      link="base_link" />
     <child
       link="FL_hip" />
@@ -196,5 +210,5 @@
       <geometry>
         <mesh
-          filename="package://go2_description/dae/FL_thigh.dae" />
+          filename="file://$(find go2_description)/dae/thigh.dae" />
       </geometry>
       <material
@@ -251,5 +265,5 @@
       <geometry>
         <mesh
-          filename="package://go2_description/dae/calf.dae" />
+          filename="file://$(find go2_description)/dae/calf.dae" />
       </geometry>
       <material
@@ -281,6 +295,6 @@
       lower="-2.7227"
       upper="-0.83776"
-      effort="35.55"
-      velocity="20.07" />
+      effort="45.43"
+      velocity="15.70" />
   </joint>
   <link
@@ -350,5 +364,5 @@
       <geometry>
         <mesh
-          filename="package://go2_description/dae/foot.dae" />
+          filename="file://$(find go2_description)/dae/foot.dae" />
       </geometry>
       <material
@@ -400,5 +414,5 @@
       <geometry>
         <mesh
-          filename="package://go2_description/dae/hip.dae" />
+          filename="file://$(find go2_description)/dae/hip.dae" />
       </geometry>
       <material
@@ -422,5 +436,5 @@
       rpy="0 0 0" />
     <parent
-      link="base" />
+      link="base_link" />
     <child
       link="FR_hip" />
@@ -455,5 +469,5 @@
       <geometry>
         <mesh
-          filename="package://go2_description/dae/thigh_mirror.dae" />
+          filename="file://$(find go2_description)/dae/thigh_mirror.dae" />
       </geometry>
       <material
@@ -510,5 +524,5 @@
       <geometry>
         <mesh
-          filename="package://go2_description/dae/calf_mirror.dae" />
+          filename="file://$(find go2_description)/dae/calf_mirror.dae" />
       </geometry>
       <material
@@ -540,6 +554,6 @@
       lower="-2.7227"
       upper="-0.83776"
-      effort="35.55"
-      velocity="20.07" />
+      effort="45.43"
+      velocity="15.70" />
   </joint>
   <link
@@ -609,5 +623,5 @@
       <geometry>
         <mesh
-          filename="package://go2_description/dae/foot.dae" />
+          filename="file://$(find go2_description)/dae/foot.dae" />
       </geometry>
       <material
@@ -659,5 +673,5 @@
       <geometry>
         <mesh
-          filename="package://go2_description/dae/hip.dae" />
+          filename="file://$(find go2_description)/dae/hip.dae" />
       </geometry>
       <material
@@ -681,5 +695,5 @@
       rpy="0 0 0" />
     <parent
-      link="base" />
+      link="base_link" />
     <child
       link="RL_hip" />
@@ -714,5 +728,5 @@
       <geometry>
         <mesh
-          filename="package://go2_description/dae/FL_thigh.dae" />
+          filename="file://$(find go2_description)/dae/thigh.dae" />
       </geometry>
       <material
@@ -769,5 +783,5 @@
       <geometry>
         <mesh
-          filename="package://go2_description/dae/calf.dae" />
+          filename="file://$(find go2_description)/dae/calf.dae" />
       </geometry>
       <material
@@ -799,6 +813,6 @@
       lower="-2.7227"
       upper="-0.83776"
-      effort="35.55"
-      velocity="20.07" />
+      effort="45.43"
+      velocity="15.70" />
   </joint>
   <link
@@ -868,5 +882,5 @@
       <geometry>
         <mesh
-          filename="package://go2_description/dae/foot.dae" />
+          filename="file://$(find go2_description)/dae/foot.dae" />
       </geometry>
       <material
@@ -918,5 +932,5 @@
       <geometry>
         <mesh
-          filename="package://go2_description/dae/hip.dae" />
+          filename="file://$(find go2_description)/dae/hip.dae" />
       </geometry>
       <material
@@ -940,5 +954,5 @@
       rpy="0 0 0" />
     <parent
-      link="base" />
+      link="base_link" />
     <child
       link="RR_hip" />
@@ -973,5 +987,5 @@
       <geometry>
         <mesh
-          filename="package://go2_description/dae/thigh_mirror.dae" />
+          filename="file://$(find go2_description)/dae/thigh_mirror.dae" />
       </geometry>
       <material
@@ -1028,5 +1042,5 @@
       <geometry>
         <mesh
-          filename="package://go2_description/dae/calf_mirror.dae" />
+          filename="file://$(find go2_description)/dae/calf_mirror.dae" />
       </geometry>
       <material
@@ -1058,6 +1072,6 @@
       lower="-2.7227"
       upper="-0.83776"
-      effort="35.55"
-      velocity="20.07" />
+      effort="45.43"
+      velocity="15.70" />
   </joint>
   <link
@@ -1127,5 +1141,5 @@
       <geometry>
         <mesh
-          filename="package://go2_description/dae/foot.dae" />
+          filename="file://$(find go2_description)/dae/foot.dae" />
       </geometry>
       <material
@@ -1179,5 +1193,5 @@
       rpy="0 0 0" />
     <parent
-      link="base" />
+      link="base_link" />
     <child
       link="imu" />
@@ -1209,5 +1223,5 @@
       rpy="0 2.8782 0" />
     <parent
-      link="base" />
+      link="base_link" />
     <child
       link="radar" />

File: go2_description/xacro/robot.xacro (robot description, xacro)
@@ -6,5 +6,5 @@
     <xacro:include filename="$(find go2_description)/xacro/leg.xacro"/>
     <!-- <xacro:include filename="$(find go2_description)/xacro/stairs.xacro"/> -->
-    <xacro:include filename="$(find go2_description)/xacro/gazebo.xacro"/>
+    <!-- <xacro:include filename="$(find go2_description)/xacro/gazebo.xacro"/> -->
     <!-- <xacro:include filename="$(find go2_gazebo)/launch/stairs.urdf.xacro"/> -->
     <!-- <xacro:stairs stairs="15" xpos="0" ypos="0" zpos="0" /> -->
